File: SolarCharger_RevC.brd (EAGLE design)
At the start: 85 x 78 mm, 123 parts, among them CON1 CON_4X200MIL, CON2 USB_BMULTICOMP, CON3 ICSP, CON4 CON_3X100MIL, CON5 CON_3X100MIL, CON6 CON_8X200MIL, CON7 CON_2X100MIL, IC1 MCP3428, IC10 S25FL208K, IC11 TPS54428, IC12 MCP14A0153, IC13 MCP14A0153, IC2 INA213LONG, IC3 MIC4605-1YM, IC4 INA213LONG, IC5 PIC18F46J50, IC6 TS6001, IC7 LMT86, IC8 24AA16, IC9 TPS62120, Q1 NX3008NBKW, Q10 NTR4101PT1G, Q11 N-FET, Q12 N-FET, Q13 N-FET, Q14 N-FET, Q15 NX3008NBKW, Q2 PSMN6R0-30YL, Q3 NX3008NBKW, Q4 NTR4101PT1G, Q5 PSMN6R0-30YL, Q6 PSMN6R0-30YL, Q7 NX3008NBKW, Q8 NX3008NBKW, Q9 NX3008NBKW, X1 ABS07-120-32.768KHZ-T, X2 ABM3-8.000MHZ-D2Y-T, X3 USB_A, X4 USB_A

Commit message: Some resistor values fixed
Parts:
- R31: value 560k -> 620k
- R32: value 270k -> 300k
- R6: value 22 -> 5R6
Changed lines of the file:
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@@
 <layer number="25" name="tNames" color="7" fill="1" visible="no" active="yes"/>
 <layer number="26" name="bNames" color="7" fill="1" visible="no" active="yes"/>
-<layer number="27" name="tValues" color="7" fill="1" visible="no" active="yes"/>
-<layer number="28" name="bValues" color="7" fill="1" visible="no" active="yes"/>
+<layer number="27" name="tValues" color="7" fill="1" visible="yes" active="yes"/>
+<layer number="28" name="bValues" color="7" fill="1" visible="yes" active="yes"/>
 <layer number="29" name="tStop" color="7" fill="3" visible="no" active="yes"/>
 <layer number="30" name="bStop" color="7" fill="6" visible="no" active="yes"/>
@@
 <element name="C17" library="00Capacitor" package="C0805" value="100n" x="67.945" y="51.435" rot="R90"/>
 <element name="Q10" library="00Mosfet" package="SOT23" value="NTR4101PT1G" x="83.185" y="53.34"/>
-<element name="R31" library="00Resistor" package="R0805" value="560k" x="80.3275" y="54.2925" rot="R90"/>
-<element name="R32" library="00Resistor" package="R0805" value="270k" x="82.8675" y="48.895" rot="R270"/>
+<element name="R31" library="00Resistor" package="R0805" value="620k" x="80.3275" y="54.2925" rot="R90"/>
+<element name="R32" library="00Resistor" package="R0805" value="300k" x="82.8675" y="48.895" rot="R270"/>
 <element name="Q1" library="00Mosfet" package="SOT23" value="NX3008NBKW" x="17.145" y="57.785" rot="R270"/>
 <element name="C5" library="00Capacitor" package="10MM" value="470u 25V" x="25.0825" y="43.815" locked="yes"/>
@@
 <element name="C7" library="00Capacitor" package="C0805" value="100n" x="25.4" y="37.465"/>
 <element name="Q3" library="00Mosfet" package="SOT23" value="NX3008NBKW" x="39.6875" y="23.495" rot="R90"/>
-<element name="R6" library="00Resistor" package="R0805" value="22" x="21.9075" y="22.225" rot="R270"/>
+<element name="R6" library="00Resistor" package="R0805" value="5R6" x="21.9075" y="22.225" rot="R270"/>
 <element name="CON3" library="00Connector" package="100MIL_6X" value="ICSP" x="89.8525" y="41.5925" rot="R90"/>
 <element name="IC5" library="00PIC" package="TQFP44" value="PIC18F46J50" x="76.2" y="41.5925" rot="R180"/>
@@
 <contactref element="L1" pad="2H"/>
 <via x="39.52875" y="33.49625" extent="1-16" drill="0.9" shape="octagon"/>
+<wire x1="29.21" y1="30.8675" x2="29.21" y2="31.0675" width="0.8128" layer="16"/>
 <wire x1="37.1475" y1="37.4775" x2="37.1475" y2="37.4775" width="0" layer="19" extent="1-16"/>
-<wire x1="29.21" y1="30.8675" x2="29.21" y2="31.0675" width="0.8128" layer="16"/>
 </signal>
 <signal name="VIN_SENSE">

Commit message: Some resistor values changed
Parts:
- R25, R27: value 25k -> 27k
Changed lines of the file:
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@@
 <element name="X4" library="00Connector" package="USB_A" value="USB_A" x="43.815" y="4.1275"/>
 <element name="R23" library="00Resistor" package="R0805" value="TBD" x="43.815" y="9.525" rot="R180"/>
-<element name="R25" library="00Resistor" package="R0805" value="25k" x="42.8625" y="12.3825" rot="R270"/>
-<element name="R27" library="00Resistor" package="R0805" value="25k" x="44.7675" y="12.3825" rot="R270"/>
+<element name="R25" library="00Resistor" package="R0805" value="27k" x="42.8625" y="12.3825" rot="R270"/>
+<element name="R27" library="00Resistor" package="R0805" value="27k" x="44.7675" y="12.3825" rot="R270"/>
 <element name="R26" library="00Resistor" package="R0805" value="68k" x="46.6725" y="10.795" rot="R270"/>
 <element name="R24" library="00Resistor" package="R0805" value="68k" x="40.9575" y="10.795" rot="R270"/>
