File: SolarCharger_RevF.brd (EAGLE design)
At the start: 85 x 78 mm, 133 parts, among them CON1 CON_4X200MIL, CON11 CON_5X100MIL, CON2 USB_BMULTICOMP, CON4 CON_3X100MIL, CON5 CON_3X100MIL, CON6 CON_8X200MIL, CON7 CON_2X100MIL, CON8 I2C, CON9 SPI, IC1 MCP3428, IC10 AT45DB321E, IC11 TPS54428, IC12 MCP14A0153, IC13 MCP14A0153, IC2 INA213, IC3 MIC4605-1YM, IC4 INA213, IC5 PIC18F47J53, IC6 TS6001, IC7 LMT86, IC8 24AA16, IC9 TPS62120, Q1 NX3008NBKW, Q10 NTR4101PT1G, Q11 N-FET, Q12 N-FET, Q13 N-FET, Q14 N-FET, Q15 NX3008NBKW, Q2 PSMN6R0-30YL, Q3 NX3008NBKW, Q4 NTR4101PT1G, Q5 PSMN6R0-30YL, Q6 PSMN6R0-30YL, Q7 NX3008NBKW, Q8 NX3008NBKW, Q9 NX3008NBKW, X1 ABS07-120-32.768KHZ-T, X2 ABM3-8.000MHZ-D2Y-T, X3 USB_A, X4 USB_A

Commit message: Revision F: Just swapped 2 signals
Parts:
- C22: value 1.8n -> 1u
- IC6: value TS6001 -> TI_REF2925
Changed lines of the file:
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@@
 <element name="C14" library="00Capacitor" package="C0805" value="100n" x="74.6125" y="32.7025" rot="R270"/>
 <element name="CON4" library="00Connector" package="100MIL_3X" value="CON_3X100MIL" x="10.16" y="46.355" rot="R90"/>
-<element name="IC6" library="00VoltageReference" package="SOT23" value="TS6001" x="69.215" y="51.435"/>
-<element name="C22" library="00Capacitor" package="C0805" value="1.8n" x="71.755" y="51.435" rot="R90"/>
+<element name="IC6" library="00VoltageReference" package="SOT23" value="TI_REF2925" x="69.215" y="51.435"/>
+<element name="C22" library="00Capacitor" package="C0805" value="1u" x="71.755" y="51.435" rot="R90"/>
 <element name="R10" library="00Resistor" package="R0805" value="300k" x="42.545" y="56.67375" rot="R90"/>
 <element name="IC8" library="00Logic" package="SOT-23-5" value="24AA16" x="76.2" y="53.6575" rot="R90"/>
