File: SolarCharger_RevF.sch (EAGLE design)
At the start: 133 parts, among them CON1 CON_4X200MIL, CON11 CON_5X100MIL, CON2 USB_BMULTICOMP, CON4 CON_3X100MIL, CON5 CON_3X100MIL, CON6 CON_8X200MIL, CON7 CON_2X100MIL, CON8 I2C, CON9 SPI, IC1 MCP3428, IC10 AT45DB321E, IC11 TPS54428, IC12 MCP14A0153, IC13 MCP14A0153, IC2 INA213, IC3 MIC4605-1YM, IC4 INA213, IC5 PIC18F47J53, IC6 TS6001, IC7 LMT86, IC8 24AA16, IC9 TPS62120, Q1 NX3008NBKW, Q10 NTR4101PT1G, Q11 N-FET, Q12 N-FET, Q13 N-FET, Q14 N-FET, Q15 NX3008NBKW, Q2 PSMN6R0-30YL, Q3 NX3008NBKW, Q4 NTR4101PT1G, Q5 PSMN6R0-30YL, Q6 PSMN6R0-30YL, Q7 NX3008NBKW, Q8 NX3008NBKW, Q9 NX3008NBKW, X1 ABS07-120-32.768KHZ-T, X2 ABM3-8.000MHZ-D2Y-T, X3 USB_A, X4 USB_A

Commit message: Revision F: Just swapped 2 signals
Parts:
- C22: value 1.8n -> 1u
- IC6: value TS6001 -> TI_REF2925
Changed lines of the file:
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@@
 <part name="P+1" library="supply1" deviceset="VCC" device=""/>
 <part name="CON4" library="00Connector" deviceset="CON_3X" device="100MIL"/>
-<part name="IC6" library="00VoltageReference" deviceset="TS6001" device=""/>
+<part name="IC6" library="00VoltageReference" deviceset="TS6001" device="" value="TI_REF2925"/>
 <part name="GND29" library="00Supply" deviceset="GND" device=""/>
 <part name="P+7" library="supply1" deviceset="VCC" device=""/>
 <part name="P+8" library="supply1" deviceset="VCC" device=""/>
-<part name="C22" library="00Capacitor" deviceset="C" device="C0805" value="1.8n"/>
+<part name="C22" library="00Capacitor" deviceset="C" device="C0805" value="1u"/>
 <part name="GND30" library="00Supply" deviceset="GND" device=""/>
 <part name="R10" library="00Resistor" deviceset="RESISTOR" device="R0805" value="300k"/>
